File: 3Dprinter-laser.kicad_pcb (KiCad board)
At the start: 2 copper layers, 13 parts, among them J1 12/24V from 3D printer, J2 FAN from 3D printer, J3 To FAN, J4 To LASER PWM/TTL, U1 L7805, U2 4N35

Commit message: fix JP1
Parts:
- moved JP1 6.35 mm to (87.6, 34.3), turned to 270 degrees
Connections:
- JP1 pad 1: Net-(J3-Pad1) -> Net-(JP1-Pad1)
- JP1 pad 2: Net-(JP1-Pad2) -> Net-(J2-Pad1)
- JP1 pad 3: Net-(J2-Pad1) -> Net-(J3-Pad1)
- R1 pad 2: Net-(JP1-Pad2) -> Net-(JP1-Pad1)
- U2 pad 3: (no net) -> Net-(U2-Pad3)
- U2 pad 6: (no net) -> Net-(U2-Pad6)
Routing:
- net Net-(JP1-Pad2): track 8.15 -> 0.00 mm
- net Net-(JP1-Pad1): track 0.00 -> 5.08 mm
- net Net-(J3-Pad1): track 13.2 -> 14.5 mm
- net Net-(J2-Pad1): track 8.67 -> 8.15 mm
- added copper zone on B.Cu, net (none)
- removed copper zone on B.Cu, net Net-(J2-Pad2)
